File: GlowBand v1.0/GlowBand.kicad_sch (KiCad schematic)
At the start: 68 parts, among them Q1 SK338P, Q2 MMBT2222A, Q3 MMBT2222A, SW1 SSAL220100, U1 AP2007SPER, U2 SN74AHCT32QPWRQ1, U3 CP2102-GMR, U4 ESP32-WROOM-32E (4MB), U5 BL1117-33CX

Commit message: started new design
Other:
- note added: "Multi cell battery management: MM3474F05VBE for controlling all batteries + MM3474 for each cell? or BQ7791504PW for each cell instead?"
- note removed: "Multi cell battery management: MM3474F05VBE for controlling all batteries + MM3474 for each cell?"
Changed lines of the file:
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@@
     (effects (font (size 3 3)) (justify left bottom))
   )
-  (text "Multi cell battery management:\n\nMM3474F05VBE for controlling all batteries + MM3474 for each cell?\n	"
+  (text "Multi cell battery management:\n\nMM3474F05VBE for controlling all batteries + MM3474 for each cell?\n\nor BQ7791504PW for each cell instead?"
     (at 95.25 400.05 0)
     (effects (font (size 1.27 1.27)) (justify left bottom))
