File: GlowBand Dock PCB/GlowBand Dock PCB.kicad_pcb (KiCad board)
At the start: 2 copper layers, 26.8 x 18.4 mm, 8 parts, among them P1 Magnetic Pogopin 6pin female, U1 UMH3N, U3 CP2102-GMR

Commit message: updated pcbs
Parts:
- added C3: 1uF, Capacitor_SMD:C_0402_1005Metric, F.Cu at (111.6, 72.4)
- added C4: 0.1uF, Capacitor_SMD:C_0402_1005Metric, F.Cu at (111.6, 71.3)
- added G***: LOGO, LOGO, B.Cu at (108.9, 69.8)
- added P2: Solder_Pad, footprint:Solder pad, F.Cu at (88.7, 70.9)
- added P3: Solder_Pad, footprint:Solder pad, F.Cu at (92.8, 70.9)
- added U2: 918-418K2022Y40003, footprint:TYPE-C-SMD_918-418K2022Y40003, F.Cu at (99.6, 70.8)
- P1: value Magnetic Pogopin 6pin female -> Magnetic_Pogopin_6pin_male; footprint footprint:Magnetic Pogopin 6pin female -> footprint:Magnetic Pogopin 6pin male
- moved P1 75.9 mm to (86.5, 58.9), turned to -90 degrees
- moved C1 56.1 mm to (109.7, 72.3), turned to -90 degrees
- moved U3 55.6 mm to (108.7, 67.2)
- moved C2 55.2 mm to (108.4, 72.9), turned to 90 degrees
- moved R2 54.9 mm to (104.8, 71.9), turned to -90 degrees
- moved R1 54.5 mm to (104.8, 69.9), turned to 90 degrees
- moved U1 54.1 mm to (108.9, 62.1), turned to 0 degrees
- moved F1 53.3 mm to (98.3, 65.8), turned to 180 degrees
Connections:
- C1 pad 1: GND -> Net-(C1-Pad1)
- C1 pad 2: +3V3 -> GND
- C2 pad 1: +3V3 -> GND
- C2 pad 2: GND -> Net-(C1-Pad1)
- F1 pad 1: unconnected-(F1-Pad1) -> Net-(F1-Pad1)
- F1 pad 2: unconnected-(F1-Pad2) -> VBUS
- U3 pad 6: +3V3 -> Net-(C1-Pad1)
- U3 pad 7: +3V3 -> VBUS
Routing:
- net GND: track 0.00 -> 46.6 mm, vias 0 -> 7
- net VBUS: track 0.00 -> 37.5 mm, vias 0 -> 2
- net USB-C DATA+: track 0.00 -> 21.6 mm, vias 0 -> 3
- net DTR: track 0.00 -> 17.2 mm, vias 0 -> 2
- net USB-C DATA-: track 0.00 -> 16.0 mm, vias 0 -> 2
- net Net-(F1-Pad1): track 0.00 -> 14.2 mm
- net RTS: track 0.00 -> 11.7 mm, vias 0 -> 2
- net USB-C CC1: track 0.00 -> 11.0 mm, vias 0 -> 2
- net RXD0: track 0.00 -> 10.3 mm, vias 0 -> 1
- net IO0: track 0.00 -> 8.04 mm
- net TXD0: track 0.00 -> 7.59 mm
- net USB-C CC2: track 0.00 -> 6.27 mm, vias 0 -> 2
- net Net-(C1-Pad1): track 0.00 -> 3.56 mm
- net EN: track 0.00 -> 2.82 mm
- net (no net): vias 0 -> 2
- added copper zone on B.Cu, net GND
- added copper zone on F.Cu, net GND
Other:
- board size 26.8 x 18.4 mm -> 26.8 x 15.4 mm
- board text added: "5V"
- board text added: "EN"
- board text added: "G"
- board text added: "GlowBand Dock PCB v1.0 beta 1"
- board text added: "IO0"
- board text added: "JLCJLCJLCJLC"
- board text added: "RX"
- board text added: "TX"
- board text added: "https:// bit.ly/ 3UXm0vi"
