File: GlowBand Dock PCB/GlowBand Dock PCB.kicad_sch (KiCad schematic)
At the start: 8 parts, among them P1 Magnetic Pogopin 6pin female, U1 UMH3N, U3 CP2102-GMR

Commit message: updated pcbs
Parts:
- removed P1: Magnetic Pogopin 6pin female, footprint:Magnetic Pogopin 6pin female, symbol MyParts:Magnetic Pogopin 6pin female
- added C3: 1uF, Capacitor_SMD:C_0402_1005Metric, symbol Device:0.1uF_0603
- added C4: 0.1uF, Capacitor_SMD:C_0402_1005Metric, symbol Device:0.1uF_0603
- added P1: Magnetic_Pogopin_6pin_male, footprint:Magnetic Pogopin 6pin male, symbol MyParts:Magnetic_Pogopin_6pin_male
- added P2, P3: Solder_Pad, footprint:Solder pad, symbol MyParts:Solder_Pad
- added U2: 918-418K2022Y40003, footprint:TYPE-C-SMD_918-418K2022Y40003, symbol MyParts:918-418K2022Y40003
Connections:
- net EN: now also P1.6
- net GND: now also C1.2, C2.1, C3.2, C4.2, P1.2, P3.1, U2.0 (EH), U2.A1 (GND), U2.A12 (GND), U2.B1 (GND), U2.B12 (GND); no longer C1.1, C2.2
- net IO0: now also P1.5
- net RXD0: now also P1.3
- net TXD0: now also P1.4
- net USB-C CC1: now also U2.A5 (CC1)
- net USB-C CC2: now also U2.B5 (CC2)
- net USB-C DATA+: now also U2.A6 (DP1), U2.B6 (DP2)
- net USB-C DATA-: now also U2.A7 (DN1), U2.B7 (DN2)
- net VBUS: now also F1.2, U3.7 (REGIN), C3.1, C4.1, P1.1, P2.1
- net at F1.1: now also U2.A4 (VBUS), U2.A9 (VBUS), U2.B4 (VBUS), U2.B9 (VBUS)
- removed net +3V3: C1.2, C2.1, U3.6 (VDD), U3.7 (REGIN)
- new net: C1.1, C2.2, U3.6 (VDD)
Other:
- note removed: "To Do: replace with male connector"
- note removed: "To Do: use REGIN via VBUS"
- moved on the sheet: C1, C2, F1, R1, R2, U3
