File: GlowBand PCB/GlowBand PCB.kicad_sch (KiCad schematic)
At the start: 74 parts, among them P1 Solder_Pad, P2 Solder_Pad, P3 Solder_Pad, P4 Solder_Pad, P5 Solder_Pad, P6 Solder_Pad, P7 Solder_Pad, P8 Solder_Pad, P9 Magnetic Pogopin 6pin female, SW1 TS24CA, SW2 TS24CA, SW3 TS-1185EC-C-D-B, SW4 TS-1185EC-C-D-B, U1 ESP32-WROOM-32E, U10 SN74LVC1G373DBVR, U13 AP40P05, U15 MSM261D4030H1CPM, U16 AP40P05, U17 AO3400A, U18 FS8205A, U19 TP4056, U2 FXL0530-6R8-M, U20 DW01A, U3 SN74LVC2T45DCUR, U4 TPS61032PWPR, U5 AP40P05, U6 SS54, U7 SPX3819M5-L-3-3_TR, U9 AP40P05

Commit message: updated pcbs
Connections:
- net +3V3: now also SW1.3, SW2.3
- net GND: no longer SW1.3, SW2.3
Changed lines of the file:
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@@
-    (pin "1")
-  )
-  (symbol (lib_id "power:GND") (at 354.33 83.82 270) (mirror x) (unit 1)
-    (in_bom yes) (on_board yes)
-    (property "Reference" "#PWR0135" (id 0) (at 347.98 83.82 0)
-      (effects (font (size 1.27 1.27)) hide)
-    )
-    (property "Value" "GND" (id 1) (at 346.71 83.82 90)
-      (effects (font (size 1.27 1.27)) (justify left))
-    )
-    (property "Footprint" "" (id 2) (at 354.33 83.82 0)
-      (effects (font (size 1.27 1.27)) hide)
-    )
-    (property "Datasheet" "" (id 3) (at 354.33 83.82 0)
-      (effects (font (size 1.27 1.27)) hide)
-    )
     (pin "1")
   )
@@
     (pin "1")
   )
-  (symbol (lib_id "power:GND") (at 354.33 97.79 270) (mirror x) (unit 1)
-    (in_bom yes) (on_board yes)
-    (property "Reference" "#PWR0136" (id 0) (at 347.98 97.79 0)
-      (effects (font (size 1.27 1.27)) hide)
-    )
-    (property "Value" "GND" (id 1) (at 346.71 97.79 90)
-      (effects (font (size 1.27 1.27)) (justify left))
-    )
-    (property "Footprint" "" (id 2) (at 354.33 97.79 0)
-      (effects (font (size 1.27 1.27)) hide)
-    )
-    (property "Datasheet" "" (id 3) (at 354.33 97.79 0)
-      (effects (font (size 1.27 1.27)) hide)
-    )
-    (pin "1")
-  )
   (symbol (lib_id "Device:R") (at 114.3 223.52 270) (unit 1)
     (in_bom yes) (on_board yes)
@@
     (property "Datasheet" "https://item.szlcsc.com/236104.html" (id 3) (at 214.63 196.85 0)
       (effects (font (size 1.27 1.27)) (justify left) hide)
-    )
-    (property "LCSC" "" (id 4) (at 205.74 199.39 0)
-      (effects (font (size 1.27 1.27)) hide)
     )
     (property "LCSC #" "C9055" (id 5) (at 205.74 199.39 0)
@@
     (pin "2")
   )
+  (symbol (lib_id "power:+3.3V") (at 354.33 83.82 90) (unit 1)
+    (in_bom yes) (on_board yes)
+    (property "Reference" "#PWR0118" (id 0) (at 358.14 83.82 0)
+      (effects (font (size 1.27 1.27)) hide)
+    )
+    (property "Value" "+3.3V" (id 1) (at 347.98 83.82 90))
+    (property "Footprint" "" (id 2) (at 354.33 83.82 0)
+      (effects (font (size 1.27 1.27)) hide)
+    )
+    (property "Datasheet" "" (id 3) (at 354.33 83.82 0)
+      (effects (font (size 1.27 1.27)) hide)
+    )
+    (pin "1")
+  )
   (symbol (lib_id "power:+3.3V") (at 287.02 227.33 270) (unit 1)
     (in_bom yes) (on_board yes)
@@
     (pin "1")
     (pin "2")
+  )
+  (symbol (lib_id "power:+3.3V") (at 354.33 97.79 90) (unit 1)
+    (in_bom yes) (on_board yes)
+    (property "Reference" "#PWR0122" (id 0) (at 358.14 97.79 0)
+      (effects (font (size 1.27 1.27)) hide)
+    )
+    (property "Value" "+3.3V" (id 1) (at 347.98 97.79 90))
+    (property "Footprint" "" (id 2) (at 354.33 97.79 0)
+      (effects (font (size 1.27 1.27)) hide)
+    )
+    (property "Datasheet" "" (id 3) (at 354.33 97.79 0)
+      (effects (font (size 1.27 1.27)) hide)
+    )
+    (pin "1")
   )
   (symbol (lib_id "power:GND") (at 85.09 198.12 270) (mirror x) (unit 1)
@@
       (reference "#PWR0117") (unit 1) (value "GND") (footprint "")
     )
+    (path "/8ee2799d-6a0d-427d-abbc-c4b49ff05d54"
+      (reference "#PWR0118") (unit 1) (value "+3.3V") (footprint "")
+    )
     (path "/c7234a7e-d638-4eef-ad28-d2bff57ab5b8"
       (reference "#PWR0119") (unit 1) (value "+5V") (footprint "")
@@
       (reference "#PWR0121") (unit 1) (value "GND") (footprint "")
     )
+    (path "/bb222cb7-fedf-4bcc-84c4-83e69c66ccbe"
+      (reference "#PWR0122") (unit 1) (value "+3.3V") (footprint "")
+    )
     (path "/b434be0c-57ff-473e-936e-4fb8a43882fb"
       (reference "#PWR0123") (unit 1) (value "+5V") (footprint "")
@@
       (reference "#PWR0134") (unit 1) (value "GND") (footprint "")
     )
-    (path "/1a15a439-c967-4867-af9f-3925c8e9f8fc"
-      (reference "#PWR0135") (unit 1) (value "GND") (footprint "")
-    )
-    (path "/2ea54bd4-1a8a-4483-a044-faae3a99b555"
-      (reference "#PWR0136") (unit 1) (value "GND") (footprint "")
-    )
     (path "/b385b09a-f424-4eaf-bade-69ba3d3b582a"

Commit message: added gyroscope to GlowBand
Parts:
- added C10, C11: 0.1uF, Capacitor_SMD:C_0402_1005Metric, symbol Device:C
- added JP2: SolderJumper_2_Bridged, Jumper:SolderJumper-2_P1.3mm_Bridged_RoundedPad1.0x1.5mm, symbol Jumper:SolderJumper_2_Bridged
- added R5, R6: 10K, Resistor_SMD:R_0402_1005Metric, symbol Device:10K 0603
- added U8: LSM6DS3TR-C, footprint:LGA-14_L3.0-W2.5-P0.50-TL, symbol MyParts:LSM6DS3TR-C
Connections:
- net 3.3V AFTER MOSFET: now also JP2.1 (A)
- net GND: now also C10.2, C11.2, U8.1 (SDO/SA0), U8.2 (SDx), U8.3 (SCx), U8.6 (GND), U8.7 (GND)
- net IO18/I2C INT1: now reaches U1.30 (IO18)
- net IO18/I2C INT1: now also U8.4 (INT1)
- net IO19/LED LETCH EN: now reaches U1.31 (IO19)
- net IO19/LED LETCH EN: now also U10.1 (LE)
- net IO21/I2C SDA: now reaches U1.33 (IO21)
- net IO21/I2C SDA: now also R5.1, U8.14 (SDA)
- net IO15/WS/TDO renamed IO15/WS/TDO
- net IO22/LED LETCH EN renamed IO22/I2C SCL
- net IO22/I2C SCL: now also R6.1, U8.13 (SCL); no longer U10.1 (LE)
- new net GYRO VDD: C10.1, C11.1, JP2.2 (B), R5.2, R6.2, U8.12 (CS), U8.5 (VDDIO), U8.8 (VDD)
Other:
- note added: "Gyroscope"
- moved on the sheet: C1, C12, C14, C15, C16, C17, C18, C19, C2, C20, C3, C4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

Commit message: updated pcb design and case prototype
Parts:
- removed C1: 10uF, Capacitor_SMD:C_0603_1608Metric, symbol Device:C
- removed C11, C2, C4: 0.1uF, Capacitor_SMD:C_0402_1005Metric, symbol Device:C
- removed C17: 1uF, Capacitor_SMD:C_0402_1005Metric, symbol Device:10uF 0603
- removed C20: 0.1uF, Capacitor_SMD:C_0402_1005Metric, symbol Device:0.1uF_0603
- removed C3: 10uF, Capacitor_SMD:C_0603_1608Metric, symbol Device:10uF 0603
- removed C5: 2.2uF, Capacitor_SMD:C_0603_1608Metric, symbol Device:0.1uF_0603
- removed C6: 220uF, Capacitor_SMD:C_1206_3216Metric, symbol Device:C
- removed F1: BSMD1812-300-16V, Fuse:Fuse_1812_4532Metric, symbol Device:Fuse
- removed JP1, JP2: SolderJumper_2_Bridged, Jumper:SolderJumper-2_P1.3mm_Bridged_RoundedPad1.0x1.5mm, symbol Jumper:SolderJumper_2_Bridged
- removed P9: Magnetic Pogopin 6pin female, footprint:Magnetic Pogopin 6pin female, symbol MyParts:Magnetic Pogopin 6pin female
- removed R1, R2: 62, Resistor_SMD:R_0402_1005Metric, symbol Device:R
- removed R14, R15, R16: 100K, Resistor_SMD:R_0402_1005Metric, symbol Device:10K 0603
- removed R17: 1K, Resistor_SMD:R_0402_1005Metric, symbol Device:1K_0603
- removed R18, R19: 220, Resistor_SMD:R_0402_1005Metric, symbol Device:10K 0603
- removed R20, R21: 10K, Resistor_SMD:R_0402_1005Metric, symbol Device:10K 0603
- removed R22: 2K, Resistor_SMD:R_0603_1608Metric_Pad0.98x0.95mm_HandSolder, symbol Device:R
- removed R23: 100, Resistor_SMD:R_0402_1005Metric, symbol Device:R
- removed R3, R4, R7: 100K, Resistor_SMD:R_0402_1005Metric, symbol Device:R
- removed R8: 160K, Resistor_SMD:R_0603_1608Metric, symbol Device:R
- removed SW4: TS-1185EC-C-D-B, footprint:SW-SMD_4P-L3.7-W3.0-P1.50-LS4.7, symbol MyParts:TS-1185EC-C-D-B
- removed TP1, TP2, TP3, TP4, TP5, TP6, TP7: TestPoint, TestPoint:TestPoint_Pad_D1.5mm, symbol Connector:TestPoint
- removed U1: ESP32-WROOM-32E, footprint:WIFI-SMD_ESP32-WROOM-32E, symbol MyParts:ESP32-WROOM-32E
- removed U10: SN74LVC1G373DBVR, footprint:SOT-23-6_L2.9-W1.6-P0.95-LS2.8-BR, symbol MyParts:SN74LVC1G373DBVR
- removed U13, U16, U9: AP40P05, footprint:SOT-23-3_L2.9-W1.3-P1.90-LS2.4-BR, symbol MyParts:AP40P05
- removed U15: MSM261D4030H1CPM, footprint:MIC-SMD_8P-L3.0-W4.0-P0.85-BL, symbol MyParts:MSM261D4030H1CPM
- removed U17: AO3400A, footprint:SOT-23-3_L2.9-W1.6-P1.90-LS2.8-BR, symbol MyParts:AO3400A
- removed U18: FS8205A, footprint:SOT-23-6_L2.9-W1.6-P0.95-LS2.8-BR, symbol FS8205A:FS8205A_C908265
- removed U19: TP4056, footprint:ESOP-8_L4.9-W3.9-P1.27-LS6.0-BL-EP, symbol MyParts:TP4056
- removed U2: FXL0530-6R8-M, footprint:IND-SMD_L5.4-W5.2_FXL0530, symbol MyParts:FXL0530-6R8-M
- removed U20: DW01A, footprint:SOT-23-6_L2.9-W1.6-P0.95-LS2.8-BL, symbol DW01A:DW01A_C351410
- removed U3: SN74LVC2T45DCUR, footprint:VSSOP-8_L2.4-W2.1-P0.50-LS3.2-BR, symbol MyParts:SN74LVC2T45DCUR
- removed U4: TPS61032PWPR, Package_SO:HTSSOP-16-1EP_4.4x5mm_P0.65mm_EP3.4x5mm_Mask2.46x2.31mm, symbol MyParts:TPS61032PWPR
- removed U6: SS54, footprint:SMA_L4.4-W2.8-LS5.4-RD, symbol MyParts:SS54
- removed U7: SPX3819M5-L-3-3_TR, footprint:SOT-23-5_L3.0-W1.7-P0.95-LS2.8-BR, symbol MyParts:SPX3819M5-L-3-3_TR
- removed U8: LSM6DS3TR-C, footprint:LGA-14_L3.0-W2.5-P0.50-TL, symbol MyParts:LSM6DS3TR-C
- added B1: LP803030, footprint:LP803030, symbol MyParts:LP803030
- added C1: 1uF, Capacitor_SMD:C_0402_1005Metric, symbol Device:10uF 0603
- added C11, C2, C4: 10uF, Capacitor_SMD:C_0603_1608Metric, symbol Device:10uF 0603
- added C13, C17: 0.1uF, Capacitor_SMD:C_0402_1005Metric, symbol Device:C
- added C3: 220uF, Capacitor_SMD:C_1206_3216Metric, symbol Device:C
- added C5: 4.7uF, Capacitor_SMD:C_0402_1005Metric, symbol Device:10uF 0603
- added C6: 47nF, Capacitor_SMD:C_0402_1005Metric, symbol Device:10uF 0603
- added L1: WPN4020H1R0MT, footprint:IND-SMD_L4.0-W4.0_SLW40XX, symbol MyParts:WPN4020H1R0MT
- added P10, P11, P12, P13, P14, P15, P16, P17, P18, P19, P20: Solder_Pad, footprint:Solder pad, symbol MyParts:Solder_Pad
- added P9: Magnetic_Pogopin_4pin_female, footprint:Magnetic Pogopin 4pin female, symbol MyParts:Magnetic_Pogopin_4pin_female
- added R1, R2, R3, R4, R7, R8: 10K, Resistor_SMD:R_0402_1005Metric, symbol Device:10K 0603
- added R10, R14, R15, R17: 100K, Resistor_SMD:R_0402_1005Metric, symbol Device:R
- added R16: 33K, Resistor_SMD:R_0402_1005Metric, symbol Device:R
- added R18: 5.1K, Resistor_SMD:R_0402_1005Metric, symbol Device:5.1K 1% 0603
- added R9: 100K, Resistor_SMD:R_0402_1005Metric, symbol Device:10K 0603
- added REF1: RT9471DGQW, footprint:RT9471_vias_in_pad, symbol MyParts:RT9471DGQW
- added U1: SN74LVC1G373DBVR, footprint:SOT-23-6_L2.9-W1.6-P0.95-LS2.8-BR, symbol MyParts:SN74LVC1G373DBVR
- added U10: MSM261D4030H1CPM, footprint:MIC-SMD_8P-L3.0-W4.0-P0.85-BL, symbol MyParts:MSM261D4030H1CPM
- added U11: SPX3819M5-L-3-3_TR, footprint:SOT-23-5_L3.0-W1.7-P0.95-LS2.8-BR, symbol MyParts:SPX3819M5-L-3-3_TR
- added U12: SK9822-EC20, footprint:LED-SMD_6P-L2.0-W2.0-P0.80-TL, symbol MyParts:SK9822-EC20
- added U13: 74LVC2G04DW-7, footprint:SOT-363_L2.0-W1.3-P0.65-LS2.1-BR, symbol MyParts:74LVC2G04DW-7
- added U2: PTVSHC3N12VU, footprint:DFN-3_L2.0-W2.0-P1.30-BR, symbol MyParts:PTVSHC3N12VU
- added U3, U7: AP40P05, footprint:SOT-23-3_L2.9-W1.3-P1.90-LS2.4-BR, symbol MyParts:AP40P05
- added U4: ESP32-S3-MINI-1-N8, footprint:ESP32-S3-MINI-1-N8, symbol MyParts:ESP32-S3-MINI-1-N8
- added U6: AO3400A, footprint:SOT-23-3_L2.9-W1.6-P1.90-LS2.8-BR, symbol MyParts:AO3400A
- added U8: SN74LVC2T45DCUR, footprint:VSSOP-8_L2.4-W2.1-P0.50-LS3.2-BR, symbol MyParts:SN74LVC2T45DCUR
- added U9: LSM6DS3TR-C, footprint:LGA-14_L3.0-W2.5-P0.50-TL, symbol MyParts:LSM6DS3TR-C
- C12: value 220uF -> 0.1uF; footprint Capacitor_SMD:C_1206_3216Metric -> Capacitor_SMD:C_0402_1005Metric; LCSC # C412252 -> C1525
- C16: LCSC # C19702 -> C96446
- C18: value 10uF -> 10nF; footprint Capacitor_SMD:C_0603_1608Metric -> Capacitor_SMD:C_0402_1005Metric; 100+ €0.0537 -> (none); LCSC # C96446 -> C15195
- C8: value 10nF -> 10uF; footprint Capacitor_SMD:C_0402_1005Metric -> Capacitor_SMD:C_0603_1608Metric; LCSC # C15195 -> C96446
- R11: value 100K -> 160K; footprint Resistor_SMD:R_0402_1005Metric -> Resistor_SMD:R_0603_1608Metric; LCSC # C25741 -> C22813
- R12: value 33K -> 100K; LCSC # C25779 -> C25741
- R13: value 100K -> 62; LCSC # C25741 -> C4962
- R5, R6: value 10K -> 100K; 100+ €0.0011 -> (none); 1000+ €0.0009 -> (none); LCSC # C25744 -> C25741
Connections:
- net IO22/I2C SCL is gone; now on net -BATT: R6.1
- net LED2 DATA OUT is gone; now on net -BATT: P5.1
- net +3V3: now also C19.2, U5.2 (S), C4.2, P17.1, R1.1, R14.2, R15.1, R18.1, R2.1, R3.1, R4.1, R9.2, U1.5 (VCC), U11.5 (OUT), U13.5 (VCC), U4.3 (3V3); no longer C9.2, SW1.3, SW2.3
- net +5V: now also C16.2, C8.2, C9.2, R5.2, L1.2, P20.1, REF1.15 (SYS), REF1.16 (SYS), U11.1 (IN), U11.3 (EN), U3.2 (S); no longer C7.2
- net +BATT: now also C7.2, R16.2, REF1.13 (BAT), REF1.14 (BAT), U7.2 (S); no longer C19.1, R12.2, U5.2 (S)
- net -BATT: now also C10.2, C12.2, C14.1, C15.1, C16.1, C18.1, C19.1, C7.1, C8.1, C9.1, P2.1, R12.1, SW1.3, SW2.3, SW3.1, C1.1, C11.1, C13.2, C17.2, C2.1, C3.2, C4.1, C5.2, P19.1, P9.4, R17.1, R8.1, REF1.17 (GND), REF1.18 (GND), REF1.25 (EP), U1.2 (GND), U10.5 (GND), U10.6 (GND), U10.7 (GND), U10.8 (GND), U11.2 (GND), U12.2 (GND), U13.2 (GND), U2.1 (A), U2.2 (1), U4.1 (GND), U4.2 (GND), U4.42 (GND), U4.43 (GND), U4.46 (GND), U4.47 (GND), U4.48 (GND), U4.49 (GND), U4.50 (GND), U4.51 (GND), U4.52 (GND), U4.53 (GND), U4.54 (GND), U4.55 (GND), U4.56 (GND), U4.57 (GND), U4.58 (GND), U4.59 (GND), U4.60 (GND), U4.61 (GND), U4.61_1 (GND), U4.61_2 (GND), U4.61_3 (GND), U4.61_4 (GND), U4.61_5 (GND), U4.61_6 (GND), U4.61_7 (GND), U4.61_8 (GND), U4.62 (GND), U4.63 (GND), U4.64 (GND), U4.65 (GND), U6.2 (S), U8.3 (A2), U8.4 (GND), U8.5 (DIR), U8.6 (B2), U9.1 (SDO/SA0), U9.2 (SDx), U9.3 (SCx), U9.6 (GND), U9.7 (GND); no longer P8.1, R13.1
- net 3.3V AFTER MOSFET: now also C12.1, C14.2, C15.2, U5.3 (D), C13.1, C17.1, P18.1, U10.1 (VDD), U8.8 (VCCB), U9.12 (CS), U9.5 (VDDIO), U9.8 (VDD)
- net 5V AFTER MOSFET: now also C10.1, P3.1, C3.1, U12.5 (VDD), U3.3 (D), U8.1 (VCCA); no longer C12.1, P1.1, P4.1
- net EN: now also SW3.2, C11.2, P14.1, R18.2, U4.45 (EN); no longer C16.2
- net LED1 DATA OUT: now also P4.1, R13.2; no longer P2.1
- net RXD0: now also P13.1, U4.40 (RXD0)
- net TXD0: now also P12.1, U4.39 (TXD0)
- net VBUS: now also C1.2, P9.3, R10.2, REF1.1 (VBUS), REF1.24 (VAC), U2.3 (K); no longer C18.1, U5.1 (G)
- net IO7/VBUS: now reaches R11.2
- net IO7/VBUS: now also R10.1, U4.11 (IO7)
- net IO8/I2C SDA: now reaches P7.1
- net IO8/I2C SDA: now also R1.2, REF1.6 (SDA), U4.12 (IO8), U9.14 (SDA)
- removed net GND: C10.2, C12.2, C14.1, C15.1, C16.1, C18.2, C19.2, C7.1, C8.1, C9.1, P3.1, P6.1, SW3.1
- removed net GYRO VDD: C10.1, R5.2, R6.2
- net IO21/I2C SDA: no longer names the net of R5.1
- net IO21/I2C SDA: now also U5.1 (G), R9.1, U3.1 (G), U6.3 (D)
- removed net IO26/BATT VOLT: R12.1, R13.2
- net IO33/MAINBUTTON: no longer names the net of SW1.4
- net IO33/MAINBUTTON: now also R14.1, U13.1 (1A)
- net IO4/BUTTON2 renamed IO0/BOOT
- net IO0/BOOT: now also R15.2, U13.3 (2A)
- new net: C2.2, REF1.23 (PMID)
- new net: C6.2, L1.1, REF1.19 (SW), REF1.20 (SW)
- new net: P1.1, U7.3 (D)
- new net: C18.2, U11.4 (BYP)
- new net: C6.1, REF1.21 (BTST)
- new net: R6.2, U1.4 (Q), U6.1 (G)
- new net: R12.2, U7.1 (G)
- new net: R13.1, U8.2 (A1)
- new net: R7.2, R8.2, REF1.11 (TS)
- new net IO0/ACTIONBUTTON: P15.1, U4.4 (IO0)
- new net IO10/I2C GRYO INT: R3.2, U4.14 (IO10), U9.4 (INT1)
- new net IO11/I2C BATT IC INT: R4.2, REF1.7 (INT#), U4.15 (IO11)
- new net IO12/I2S WS: U10.2 (L/R), U4.16 (IO12)
- new net IO13/I2S SCK: U10.3 (CLK), U4.17 (IO13)
- new net IO14/I2S SD: U10.4 (DATA), U4.18 (IO14)
- new net IO15/LED LETCH EN: U1.1 (LE), U4.19 (IO15)
- new net IO16/POWERMOSFETS: U1.3 (D), U4.20 (IO16)
- new net IO1/POWERBUTTON: P16.1, U13.6 (1Y), U4.5 (IO1)
- new net IO2/BATT VOLT: R16.1, R17.2, U4.6 (IO2)
- new net IO35/SPI MO: P11.1, U4.31 (IO35)
- new net IO36/SPI SCK: P8.1, U4.32 (IO36)
- new net IO37/SPI MI: P10.1, U4.33 (IO37)
- new net IO39/STATUS LED CLOCK: U12.4 (CKL), U4.35 (IO39)
- new net IO3/ACTIONBUTTON: U13.4 (2Y)
- new net IO4: U4.8 (IO4)
- new net IO40/STATUS LED DATA: U12.3 (SDI), U4.36 (IO40)
- new net IO41/LED2: U4.37 (IO41)
- new net IO42/LED1: U4.38 (IO42), U8.7 (B1)
- new net IO47/BATT IC EN: REF1.9 (CE#), U4.27 (IO47)
- new net IO5: U4.9 (IO5)
- new net IO6: U4.10 (IO6)
- new net IO9/I2C SCL: P6.1, R2.2, REF1.5 (SCL), U4.13 (IO9), U9.13 (SCL)
- new net REGN: C5.1, R7.1, REF1.22 (REGN)
- new net USB D+: P9.1, U4.24 (IO20)
- new net USB D-: P9.2, U4.23 (IO19)
- no-connect marks 0 -> 27
Other:
- note added: "Battery"
- note added: "Dock connector"
- note added: "LED strip pads"
- note added: "Lipo charging & protection & 5V converter"
- note added: "Pads"
- note added: "Status LED"
- note removed: "5V converter"
- note removed: "LED strip connectors"
- note removed: "Lipo charging & protection"
- note removed: "Pins 12,13,14,15 for JTAG debugger"
- note removed: "Pins IN/OUT"
- note removed: "Power"
- note removed: "Power Saving mode is on (SYNC low)"
- note removed: "Programm charging speed with resistor: 10K => 130 mA 5K => 250mA 4K => 300mA 3K => 400mA 2K => 580mA 1.66K => 690mA 1.5K => 780mA 1.33K => 900mA 1.2K => 1000mA"
- note removed: "Reset"
- note removed: "USB-C dock connector"
